File: PCB/Groupe 2 final PCB.sch (EAGLE design)
At the start: 19 parts, among them IC1 4511N, IC2 4511N, IC3 PIC16F877P

Commit message: Final Board
Parts:
- renumbered C1 to C1-15PF, C2 to C2-15PF, C3 to C3-680NF, IC1 to 4511N-D, IC2 to 4511N-U, R2 to R2-1K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
